Commit message: adjust x2 config

File: source/whole_body_tracking/whole_body_tracking/assets/x2/x2_ultra_simple_collision_23dof.urdf (robot description, URDF)
Before this commit: robot x2, 39 links, 38 joints
Joints:
- joint left_wrist_pitch_joint: type revolute -> fixed
- joint left_wrist_roll_joint: type revolute -> fixed
- joint left_wrist_yaw_joint: type revolute -> fixed
- joint right_wrist_pitch_joint: type revolute -> fixed
- joint right_wrist_roll_joint: type revolute -> fixed
- joint right_wrist_yaw_joint: type revolute -> fixed
