Commit message: x2 sim2sim, fix extra dofs

File: source/whole_body_tracking/whole_body_tracking/assets/x2/x2_ultra_simple_collision.urdf (robot description, URDF)
Before this commit: robot x2t2.5, 39 links, 38 joints
Joints:
- joint head_pitch_joint: type revolute -> fixed
- joint head_yaw_joint: type revolute -> fixed
- joint left_wrist_pitch_joint: type revolute -> fixed
- joint left_wrist_roll_joint: type revolute -> fixed
- joint left_wrist_yaw_joint: type revolute -> fixed
- joint right_wrist_pitch_joint: type revolute -> fixed
- joint right_wrist_roll_joint: type revolute -> fixed
- joint right_wrist_yaw_joint: type revolute -> fixed

Commit message: back to 29 dof

File: source/whole_body_tracking/whole_body_tracking/assets/x2/x2_ultra_simple_collision.urdf (robot description, URDF)
Before this commit: robot x2, 39 links, 38 joints
Joints:
- joint left_wrist_pitch_joint: type fixed -> revolute
- joint left_wrist_roll_joint: type fixed -> revolute
- joint left_wrist_yaw_joint: type fixed -> revolute
- joint right_wrist_pitch_joint: type fixed -> revolute
- joint right_wrist_roll_joint: type fixed -> revolute
- joint right_wrist_yaw_joint: type fixed -> revolute
